File: Accio.sch (KiCad schematic (older format))
At the start: 18 parts, among them J1 Conn_01x02, J2 Conn_02x04_Counter_Clockwise, J3 Conn_01x03, Q1 BC547, U1 LM1117-3.3

Commit message: Add files via upload
Parts:
- removed J2: Conn_02x04_Counter_Clockwise, Pin_Headers:Pin_Header_Angled_2x04_Pitch2.54mm, symbol Conn_02x04_Counter_Clockwise
- added J2: Conn_02x04_Odd_Even, Pin_Headers:Pin_Header_Straight_2x04_Pitch2.54mm, symbol Conn_02x04_Odd_Even
- added J4, J5: Conn_01x03, Pin_Headers:Pin_Header_Straight_1x03_Pitch2.54mm, symbol Conn_01x03
- J1: footprint Pin_Headers:Pin_Header_Angled_1x02_Pitch2.54mm -> Pin_Headers:Pin_Header_Straight_1x02_Pitch2.54mm
- J3: footprint Pin_Headers:Pin_Header_Angled_1x03_Pitch2.54mm -> Pin_Headers:Pin_Header_Straight_1x03_Pitch2.54mm
Connections:
- net ESP_RX: now also J2.8 (Pin_8)
- net ESP_TX: now also J2.1 (Pin_1)
- net GND: now also J2.2 (Pin_2), J4.1 (Pin_1), J4.2 (Pin_2), J4.3 (Pin_3), J5.3 (Pin_3)
- net GPIO0: now also J2.6 (Pin_6), J5.2 (Pin_2); no longer R4.1
- net GPIO2: now also R4.1, J2.4 (Pin_4)
- net Vdd_ESP: now also J2.3 (Pin_3), J2.5 (Pin_5), J2.7 (Pin_7), J5.1 (Pin_1)
- no-connect marks 2 -> 0
Other:
- moved on the sheet: C1, C2, C4, D1, J1, R1, U1
