File: Accio.kicad_pcb (KiCad board)
At the start: 2 copper layers, 59.7 x 59.7 mm, 20 parts, among them J1 Conn_01x02, J2 Conn_02x04_Odd_Even, J3 Conn_01x03, J4 Conn_01x03, J5 Conn_01x03, Q1 BC547, U1 LM1117-3.3

Commit message: Add files via upload
Parts:
- added J6: Conn_01x03, Pin_Headers:Pin_Header_Straight_1x03_Pitch2.54mm, F.Cu at (99.0, 53.0)
- added J7: Conn_01x03, Pin_Headers:Pin_Header_Straight_1x03_Pitch2.54mm, F.Cu at (78.0, 36.0)
Connections:
- J2 pad 5: /Vdd_ESP -> /Reset
Routing:
- net /Vdd_ESP: track 107.9 -> 149.5 mm, vias 4 -> 7
- net /GPIO2: track 30.7 -> 69.5 mm, vias 1 -> 4
- net GND: track 200.8 -> 224.8 mm
- net /Reset: track 0.00 -> 23.4 mm, vias 0 -> 1
